File: hardware/Zvonek/Zvonek.brd (EAGLE design)
At the start: 36.8 x 28.9 mm, 34 parts, among them J1 J25MM, K1 ARK500/3, T1 BC847, T2 BC847, T3 BC847, T4 BC847, T5 IRF9530

Commit message: Change some component values
This version matches the board that was manufactured.
Parts:
- R5: value 10k -> 100k
- R8: value 10k -> 33k
Changed lines of the file:
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@@
 <attribute name="VALUE" x="12.7" y="16.51" size="1.27" layer="28" rot="MR270"/>
 </element>
-<element name="R8" library="rcl" library_urn="urn:adsk.eagle:library:334" package="R1206" package3d_urn="urn:adsk.eagle:package:23540/2" value="10k" x="15.24" y="13.97" smashed="yes" rot="MR0">
+<element name="R8" library="rcl" library_urn="urn:adsk.eagle:library:334" package="R1206" package3d_urn="urn:adsk.eagle:package:23540/2" value="33k" x="15.24" y="13.97" smashed="yes" rot="MR0">
 <attribute name="NAME" x="16.51" y="15.24" size="1.27" layer="26" rot="MR0"/>
 <attribute name="POPULARITY" value="41" x="-26.67" y="-10.16" size="1.778" layer="28" rot="MR0" display="off"/>
@@
 <attribute name="VALUE" x="16.51" y="11.43" size="1.27" layer="28" rot="MR0"/>
 </element>
-<element name="R5" library="rcl" library_urn="urn:adsk.eagle:library:334" package="R1206" package3d_urn="urn:adsk.eagle:package:23540/2" value="10k" x="29.21" y="24.13" smashed="yes" rot="MR0">
+<element name="R5" library="rcl" library_urn="urn:adsk.eagle:library:334" package="R1206" package3d_urn="urn:adsk.eagle:package:23540/2" value="100k" x="29.21" y="24.13" smashed="yes" rot="MR0">
 <attribute name="NAME" x="30.48" y="25.4" size="1.27" layer="26" rot="MR0"/>
 <attribute name="POPULARITY" value="41" x="13.97" y="-6.35" size="1.778" layer="28" rot="MR0" display="off"/>
@@
 <wire x1="22.86" y1="19.05" x2="24.13" y2="19.05" width="1.5" layer="16"/>
 <wire x1="22.73" y1="24.13" x2="22.225" y2="23.625" width="1.5" layer="16"/>
-<wire x1="22.225" y1="23.625" x2="22.225" y2="19.05" width="1.5" layer="16"/>
+<wire x1="22.225" y1="19.05" x2="22.225" y2="23.625" width="1.5" layer="16"/>
 <wire x1="24.13" y1="19.05" x2="24.511" y2="19.431" width="1.5" layer="16"/>
 <wire x1="24.511" y1="19.431" x2="25.756" y2="19.431" width="1.5" layer="16"/>
